File: Floppy Disk Controller.kicad_pcb (KiCad board)
At the start: 2 copper layers, 81.3 x 40 mm, 15 parts, among them J1 Interis_Expansion_PCBEdge, J2 Conn_02x17_Odd_Even, U1 74LS125, U2 74LS138, U3 WD37C65C, X1 16 MHz

Commit message: Updated schematic
Parts:
- removed JP1, JP2: Jumper_3_Bridged12, Connector_PinHeader_2.54mm:PinHeader_1x03_P2.54mm_Vertical
- moved X1 2.54 mm to (137.2, 108.0)
Connections:
- net FDC_CCR renamed FDC_LDCR
- net PORT04 renamed PORT02
- R3 pad 2: ~{DACK} -> PORT00
- U1 pad 4: FDC_DOR -> (no net)
- U1 pad 5: ~{RD} -> (no net)
- U1 pad 6: Net-(JP2-Pad1) -> (no net)
- U1 pad 8: Net-(JP1-Pad1) -> TC
- U2 pad 9: FDC_DOR -> FDC_LDOR
- U3 pad 17: FDC_DOR -> FDC_LDOR
- U3 pad 5: ~{DACK} -> PORT00
Routing:
- net FDC_LDOR: track 0.00 -> 65.8 mm, vias 0 -> 2
- net FDC_DOR: track 65.8 -> 0.00 mm, vias 2 -> 0
- net ~{DACK}: track 64.6 -> 0.00 mm, vias 1 -> 0
- net PORT00: track 78.6 -> 29.8 mm, vias 2 -> 1
- net Net-(JP2-Pad1): track 37.2 -> 0.00 mm, vias 5 -> 0
- net Net-(JP1-Pad1): track 6.12 -> 0.00 mm
- net +5V: track 236.2 -> 231.0 mm
- net TC: track 74.2 -> 72.2 mm, vias 3 -> 4
- net Net-(U3-CLK1): track 31.8 -> 31.0 mm
Other:
- board size 81.3 x 40 mm -> 78.1 x 40 mm
- board text added: "PCB3D_BR_FDC"
- board text added: "PCB3D_TL_FDC"
