File: Floppy Disk Controller.kicad_sch (KiCad schematic)
At the start: 15 parts, among them J1 Interis_Expansion_PCBEdge, J2 Conn_02x17_Odd_Even, U1 74LS125, U2 74LS138, U3 WD37C65C, X1 16 MHz

Commit message: Updated schematic
Parts:
- removed JP1, JP2: Jumper_3_Bridged12, Connector_PinHeader_2.54mm:PinHeader_1x03_P2.54mm_Vertical, symbol Jumper:Jumper_3_Bridged12
- removed unit 2 of U1
Connections:
- net ~{DACK} is gone; now on net PORT00: R3.2, U3.5 (~{DACK})
- net TC: now also U1.8
Other:
- moved on the sheet: R2, R3, X1
